File: PCB/lagom.kicad_sch (KiCad schematic)
At the start: 159 parts, among them J1 Conn_01x04, J2 Conn_01x03, SW83 RotaryEncoder_Switch, SW84 RotaryEncoder_Switch, U1 ProMicro, U2 74HC138, U3 74HC138

Commit message: Change promicro symbol to local and remove dependency of keebio sym lib
Parts:
- U1: symbol keebio:ProMicro -> lagom:ProMicro
Changed lines of the file:
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@@
 	)
 	(symbol
-		(lib_id "keebio:ProMicro")
+		(lib_id "lagom:ProMicro")
 		(at 68.58 181.61 0)
 		(unit 1)
@@
 		(fields_autoplaced yes)
 		(property "Reference" "U1"
-			(at 68.58 158.877 0)
+			(at 68.58 160.02 0)
 			(effects
 				(font
@@
 		)
 		(property "Value" "ProMicro"
-			(at 68.58 162.687 0)
+			(at 68.58 162.56 0)
 			(effects
 				(font

Commit message: Schematic - Diode fp -> SMD MiniMELF
Parts:
- D1: footprint Button_Switch_THT:SW_PUSH_1P1T_6x3.5mm_H5.0_APEM_MJTP1250 -> Diode_SMD:D_MiniMELF
- D10, D11, D12, D13, D14, D15, D16, D17, D18, D19, D2, D20, D21, D22, D23, D24, D25, D26, D27, D28, D29, D3, D30, D31, D32, D33, D34, D35, D36, D37, D38, D39, D4, D40, D41, D42, D43, D44, D45, D46, D47, D48, D49, D5, D50, D51, D52, D53, D54, D55, D56, D57, D58, D59, D6, D60, D61, D62, D63, D64, D65, D66, D67, D68, D69, D7, D70, D71, D72, D73, D74, D8, D9: footprint Diode_THT:D_DO-34_SOD68_P7.62mm_Horizontal -> Diode_SMD:D_MiniMELF

Commit message: Layout - Complete rework
Parts:
- removed SW_ENC1, SW_ENC2: KEYSW, kailh_hotswap:SW_Kailh_HotSwap_1.00u_PCB, symbol Switch:SW_Push
- D1, D10, D11, D12, D13, D14, D15, D16, D17, D18, D19, D2, D20, D21, D22, D23, D24, D25, D26, D27, D28, D29, D3, D30, D31, D32, D33, D34, D35, D36, D37, D38, D39, D4, D40, D41, D42, D43, D44, D45, D46, D47, D48, D49, D5, D50, D51, D52, D53, D54, D55, D56, D57, D58, D59, D6, D60, D61, D62, D63, D64, D65, D66, D67, D68, D69, D7, D70, D71, D72, D73, D74, D8, D9: footprint Diode_SMD:D_MiniMELF -> lagom:D_MiniMELF_noSilk
- SW83, SW84: footprint Keebio-Parts:RotaryEncoder_EC11 -> Rotary_Encoder:RotaryEncoder_Alps_EC11E-Switch_Vertical_H20mm
- SW_6.25U_SPACE1: footprint kailh_hotswap:SW_Kailh_HotSwap_6.25u_PCB -> kailh_hotswap:SW_Kailh_HotSwap_6.25u_PCB_reverse
- SW_SPL_SPACE_L1: footprint kailh_hotswap:SW_Kailh_HotSwap_2.25u_PCB -> kailh_hotswap:SW_Kailh_HotSwap_2.25u_PCB_reverse
- SW_SPL_SPACE_R1: footprint kailh_hotswap:SW_Kailh_HotSwap_2.75u_PCB -> kailh_hotswap:SW_Kailh_HotSwap_2.75u_PCB_reverse
- U1: footprint Keebio-Parts:ArduinoProMicro-ZigZag -> lagom:ArduinoProMicro-ZigZag
- U2, U3: footprint Package_SO:TSSOP-16_4.4x5mm_P0.65mm -> Package_SO:SOIC-16_3.9x9.9mm_P1.27mm
Connections:
- net RotB: now also SW_HOME1.2
- net col6: now also SW_SPL_SPACE_M1.1; no longer SW_SPL_SPACE_M1.2
- net col9: now also SW_L1.2
- net at D68.1 (K), SW_6.25U_SPACE1.1: now also SW_SPL_SPACE_M1.2; no longer SW_SPL_SPACE_M1.1

Commit message: Add alternative LEDs instead of OLED
Parts:
- removed D14, D30: 1N4148, lagom:D_MiniMELF_noSilk, symbol Device:D_Small
- added D75: red, LED_SMD:LED_1206_3216Metric, symbol Device:LED_Small
- added D76: green, LED_SMD:LED_1206_3216Metric, symbol Device:LED_Small
- added R1, R2: 680R, Resistor_SMD:R_1206_3216Metric, symbol Device:R_Small
Connections:
- net SCL: now also D75.1 (K)
- net SDA: now also D76.1 (K)
- net VCC: now also R1.1, R2.1
- new net: D76.2 (A), R1.2
- new net: D75.2 (A), R2.2
- no-connect marks 5 -> 3
Other:
- moved on the sheet: J1
