File: PCB/lagom.kicad_pcb (KiCad board)
At the start: 2 copper layers, 305.6 x 121.8 mm, 166 parts, among them J1 Conn_01x04, J2 Conn_01x03, SW83 RotaryEncoder_Switch, SW84 RotaryEncoder_Switch, U1 ProMicro, U2 74HC138, U3 74HC138

Commit message: Layout - Complete rework
Parts:
- removed REF** (x11): MountingHole_2.2mm_M2, MountingHole:MountingHole_2.2mm_M2
- removed SW_ENC1, SW_ENC2: KEYSW, Button_Switch_Keyboard:SW_Cherry_MX_1.00u_PCB
- removed SW_LSHF1: KEYSW, Button_Switch_Keyboard:SW_Cherry_MX_2.25u_PCB
- added BT1: Battery_Cell, Connector_JST:JST_PH_S2B-PH-K_1x02_P2.00mm_Horizontal, B.Cu at (73.3, 49.1)
- added SW_ISO_LSHF1: KEYSW, kailh_hotswap:SW_Kailh_HotSwap_1.25u_PCB, F.Cu at (67.0, 123.8)
- added SW_ISO_`1: KEYSW, kailh_hotswap:SW_Kailh_HotSwap_1.00u_PCB, F.Cu at (88.5, 123.8)
- added SW_PW1: SW_SPDT, Connector_PinHeader_2.54mm:PinHeader_1x03_P2.54mm_Vertical, B.Cu at (58.2, 52.6)
- added SW_RST1: KEYSW, Button_Switch_THT:SW_PUSH_1P1T_6x3.5mm_H5.0_APEM_MJTP1250, F.Cu at (62.7, 46.9)
- C1, C2: footprint Capacitor_THT:C_Disc_D4.7mm_W2.5mm_P5.00mm -> Capacitor_SMD:C_0805_2012Metric
- D1, D10, D11, D12, D13, D14, D15, D16, D17, D18, D19, D2, D20, D21, D22, D23, D24, D25, D26, D27, D28, D29, D3, D30, D31, D32, D33, D34, D35, D36, D37, D38, D39, D4, D40, D41, D42, D43, D44, D45, D46, D47, D48, D49, D5, D50, D51, D52, D53, D54, D55, D56, D57, D58, D59, D6, D60, D61, D62, D63, D64, D65, D66, D67, D68, D69, D7, D70, D71, D72, D73, D74, D8, D9: value D_Small -> 1N4148; footprint Diode_THT:D_DO-34_SOD68_P7.62mm_Horizontal -> lagom:D_MiniMELF_noSilk
- SW83, SW84: footprint Keebio-Parts:RotaryEncoder_EC11 -> Rotary_Encoder:RotaryEncoder_Alps_EC11E-Switch_Vertical_H20mm
- SW_/1, SW_0, SW_1, SW_2, SW_3, SW_4, SW_5, SW_6, SW_7, SW_8, SW_9, SW_A1, SW_B1, SW_C1, SW_COMMA1, SW_D1, SW_DOT1, SW_DOWN1, SW_E1, SW_END1, SW_EQUAL1, SW_ESC1, SW_F1, SW_G1, SW_H1, SW_HOME1, SW_I1, SW_ISO_\1, SW_J1, SW_K1, SW_L1, SW_LEFT1, SW_LSQBR1, SW_M1, SW_MINUS1, SW_N1, SW_O1, SW_P1, SW_PGDN1, SW_PGUP1, SW_Q1, SW_QUOTE1, SW_R1, SW_RIGHT1, SW_RSQBR1, SW_S1, SW_SEMICOLON1, SW_T1, SW_U1, SW_UP1, SW_V1, SW_W1, SW_X1, SW_Y1, SW_Z1: footprint Button_Switch_Keyboard:SW_Cherry_MX_1.00u_PCB -> kailh_hotswap:SW_Kailh_HotSwap_1.00u_PCB
- SW_6.25U_SPACE1: footprint Button_Switch_Keyboard:SW_Cherry_MX_6.25u_PCB -> kailh_hotswap:SW_Kailh_HotSwap_6.25u_PCB_reverse
- SW_BCKSP1: footprint Button_Switch_Keyboard:SW_Cherry_MX_2.00u_PCB -> kailh_hotswap:SW_Kailh_HotSwap_2.00u_PCB
- SW_CAPS1, SW_RSHIFT1: footprint Button_Switch_Keyboard:SW_Cherry_MX_1.75u_PCB -> kailh_hotswap:SW_Kailh_HotSwap_1.75u_PCB
- SW_ISO_ENT1: footprint Button_Switch_Keyboard:SW_Cherry_MX_ISOEnter_PCB_Flipped_Rotated -> kailh_hotswap:SW_Kailh_HotSwap_ISOEnter_PCB
- SW_LALT_1.25U1, SW_LCMD_1.25U1, SW_LCTRL_1.25U1, SW_R_CMD1, SW_R_CTRL_1.25U1, SW_SPL_SPACE_M1: footprint Button_Switch_Keyboard:SW_Cherry_MX_1.25u_PCB -> kailh_hotswap:SW_Kailh_HotSwap_1.25u_PCB
- SW_SPL_SPACE_L1: footprint Button_Switch_Keyboard:SW_Cherry_MX_2.25u_PCB -> kailh_hotswap:SW_Kailh_HotSwap_2.25u_PCB_reverse
- SW_SPL_SPACE_R1: footprint Button_Switch_Keyboard:SW_Cherry_MX_2.75u_PCB -> kailh_hotswap:SW_Kailh_HotSwap_2.75u_PCB_reverse
- SW_TAB1: footprint Button_Switch_Keyboard:SW_Cherry_MX_1.50u_PCB -> kailh_hotswap:SW_Kailh_HotSwap_1.50u_PCB
- U1: footprint Keebio-Parts:ArduinoProMicro-ZigZag -> lagom:ArduinoProMicro-ZigZag
- U2, U3: footprint Package_DIP:DIP-16_W7.62mm_Socket -> Package_SO:SOIC-16_3.9x9.9mm_P1.27mm
- moved C2 16.3 mm to (106.7, 43.6), turned to 180 degrees
- moved D72 16.0 mm to (265.0, 55.3)
- moved D1 13.5 mm to (117.0, 48.2)
- moved D11 13.5 mm to (226.8, 48.2)
- moved D13 13.5 mm to (250.7, 48.2)
- moved D3 13.5 mm to (140.8, 48.2)
- moved D5 13.5 mm to (162.3, 48.2)
- moved D7 13.5 mm to (183.8, 48.2)
- moved D9 13.5 mm to (205.3, 48.2)
- moved D69 13.5 mm to (214.9, 57.7)
- moved D64 13.5 mm to (126.5, 57.7)
- moved D66 13.5 mm to (150.4, 57.7)
- moved D67 13.5 mm to (171.9, 57.7)
- moved D68 13.5 mm to (193.4, 57.7)
- moved D70 13.5 mm to (236.3, 57.7)
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Connections:
- D1 pad 1: Net-(D1-Pad1) -> Net-(D1-K)
- D10 pad 1: Net-(D10-Pad1) -> Net-(D10-K)
- D11 pad 1: Net-(D11-Pad1) -> Net-(D11-K)
- D12 pad 1: Net-(D12-Pad1) -> Net-(D12-K)
- D13 pad 1: Net-(D13-Pad1) -> Net-(D13-K)
- D14 pad 1: Net-(D14-Pad1) -> unconnected-(D14-K-Pad1)
- D15 pad 1: Net-(D15-Pad1) -> Net-(D15-K)
- D16 pad 1: Net-(D16-Pad1) -> Net-(D16-K)
- D17 pad 1: Net-(D17-Pad1) -> Net-(D17-K)
- D18 pad 1: Net-(D18-Pad1) -> Net-(D18-K)
- D19 pad 1: Net-(D19-Pad1) -> Net-(D19-K)
- D2 pad 1: Net-(D2-Pad1) -> Net-(D2-K)
- D20 pad 1: Net-(D20-Pad1) -> Net-(D20-K)
- D21 pad 1: Net-(D21-Pad1) -> Net-(D21-K)
- D22 pad 1: Net-(D22-Pad1) -> Net-(D22-K)
- D23 pad 1: Net-(D23-Pad1) -> Net-(D23-K)
- D24 pad 1: Net-(D24-Pad1) -> Net-(D24-K)
- D25 pad 1: Net-(D25-Pad1) -> Net-(D25-K)
- D26 pad 1: Net-(D26-Pad1) -> Net-(D26-K)
- D27 pad 1: Net-(D27-Pad1) -> Net-(D27-K)
- D28 pad 1: Net-(D28-Pad1) -> Net-(D28-K)
- D29 pad 1: Net-(D29-Pad1) -> Net-(D29-K)
- D3 pad 1: Net-(D3-Pad1) -> Net-(D3-K)
- D30 pad 1: Net-(D30-Pad1) -> unconnected-(D30-K-Pad1)
- D31 pad 1: Net-(D31-Pad1) -> Net-(D31-K)
- D33 pad 1: Net-(D33-Pad1) -> Net-(D33-K)
- D34 pad 1: Net-(D34-Pad1) -> Net-(D34-K)
- D35 pad 1: Net-(D35-Pad1) -> Net-(D35-K)
- D36 pad 1: Net-(D36-Pad1) -> Net-(D36-K)
- D37 pad 1: Net-(D37-Pad1) -> Net-(D37-K)
- D38 pad 1: Net-(D38-Pad1) -> Net-(D38-K)
- D39 pad 1: Net-(D39-Pad1) -> Net-(D39-K)
- D4 pad 1: Net-(D4-Pad1) -> Net-(D4-K)
- D40 pad 1: Net-(D40-Pad1) -> Net-(D40-K)
- D41 pad 1: Net-(D41-Pad1) -> Net-(D41-K)
- D42 pad 1: Net-(D42-Pad1) -> Net-(D42-K)
- D43 pad 1: Net-(D43-Pad1) -> Net-(D43-K)
- D44 pad 1: Net-(D44-Pad1) -> Net-(D44-K)
- D45 pad 1: Net-(D45-Pad1) -> Net-(D45-K)
- D46 pad 1: Net-(D46-Pad1) -> Net-(D46-K)
- D47 pad 1: Net-(D47-Pad1) -> Net-(D47-K)
- D49 pad 1: Net-(D49-Pad1) -> Net-(D49-K)
- D5 pad 1: Net-(D5-Pad1) -> Net-(D5-K)
- D50 pad 1: Net-(D50-Pad1) -> Net-(D50-K)
- D51 pad 1: Net-(D51-Pad1) -> Net-(D51-K)
- D54 pad 1: Net-(D54-Pad1) -> Net-(D54-K)
- D55 pad 1: Net-(D55-Pad1) -> Net-(D55-K)
- D56 pad 1: Net-(D56-Pad1) -> Net-(D56-K)
- D57 pad 1: Net-(D57-Pad1) -> Net-(D57-K)
- D58 pad 1: Net-(D58-Pad1) -> Net-(D58-K)
- D59 pad 1: Net-(D59-Pad1) -> Net-(D59-K)
- D6 pad 1: Net-(D6-Pad1) -> Net-(D6-K)
- D60 pad 1: Net-(D60-Pad1) -> Net-(D60-K)
- D61 pad 1: Net-(D61-Pad1) -> Net-(D61-K)
- D62 pad 1: Net-(D62-Pad1) -> Net-(D62-K)
- D63 pad 1: Net-(D63-Pad1) -> Net-(D63-K)
- D64 pad 1: Net-(D64-Pad1) -> Net-(D64-K)
- D65 pad 1: Net-(D65-Pad1) -> Net-(D65-K)
- D66 pad 1: Net-(D66-Pad1) -> Net-(D66-K)
- D67 pad 1: Net-(D67-Pad1) -> Net-(D67-K)
- D68 pad 1: Net-(D68-Pad1) -> Net-(D68-K)
- D69 pad 1: Net-(D69-Pad1) -> Net-(D69-K)
- D7 pad 1: Net-(D7-Pad1) -> Net-(D7-K)
- D70 pad 1: Net-(D70-Pad1) -> Net-(D70-K)
- D71 pad 1: Net-(D71-Pad1) -> Net-(D71-K)
- D72 pad 1: Net-(D72-Pad1) -> Net-(D72-K)
- D73 pad 1: Net-(D73-Pad1) -> Net-(D73-K)
- D74 pad 1: Net-(D74-Pad1) -> Net-(D74-K)
- D8 pad 1: Net-(D8-Pad1) -> Net-(D8-K)
- D9 pad 1: Net-(D9-Pad1) -> Net-(D9-K)
- SW_/1 pad 1: col11 -> Net-(D49-K)
- SW_/1 pad 2: Net-(D49-Pad1) -> col11
- SW_0 pad 1: col10 -> Net-(D11-K)
- SW_0 pad 2: Net-(D11-Pad1) -> col10
- SW_1 pad 1: col1 -> Net-(D2-K)
- SW_1 pad 2: Net-(D2-Pad1) -> col1
- SW_2 pad 1: col2 -> Net-(D3-K)
- SW_2 pad 2: Net-(D3-Pad1) -> col2
- SW_3 pad 1: col3 -> Net-(D4-K)
- SW_3 pad 2: Net-(D4-Pad1) -> col3
- SW_4 pad 1: col4 -> Net-(D5-K)
- SW_4 pad 2: Net-(D5-Pad1) -> col4
- SW_5 pad 1: col5 -> Net-(D6-K)
- SW_5 pad 2: Net-(D6-Pad1) -> col5
- SW_6 pad 1: col6 -> Net-(D7-K)
- SW_6 pad 2: Net-(D7-Pad1) -> col6
- SW_6.25U_SPACE1 pad 1: col6 -> Net-(D68-K)
- SW_6.25U_SPACE1 pad 2: Net-(D68-Pad1) -> col6
- SW_7 pad 1: col7 -> Net-(D8-K)
- SW_7 pad 2: Net-(D8-Pad1) -> col7
- SW_8 pad 1: col8 -> Net-(D9-K)
- SW_8 pad 2: Net-(D9-Pad1) -> col8
- SW_9 pad 1: col9 -> Net-(D10-K)
- SW_9 pad 2: Net-(D10-Pad1) -> col9
- SW_A1 pad 1: col1 -> Net-(D36-K)
- SW_A1 pad 2: Net-(D36-Pad1) -> col1
- SW_B1 pad 1: col6 -> Net-(D58-K)
- SW_B1 pad 2: Net-(D58-Pad1) -> col6
- SW_BCKSP1 pad 1: col14 -> Net-(D15-K)
- SW_BCKSP1 pad 2: Net-(D15-Pad1) -> col14
- SW_C1 pad 1: col4 -> Net-(D56-K)
- SW_C1 pad 2: Net-(D56-Pad1) -> col4
- SW_CAPS1 pad 1: col0 -> Net-(D35-K)
- SW_CAPS1 pad 2: Net-(D35-Pad1) -> col0
- SW_COMMA1 pad 1: col9 -> Net-(D61-K)
- SW_COMMA1 pad 2: Net-(D61-Pad1) -> col9
- SW_D1 pad 1: col3 -> Net-(D38-K)
- SW_D1 pad 2: Net-(D38-Pad1) -> col3
- SW_DOT1 pad 1: col10 -> Net-(D62-K)
- SW_DOT1 pad 2: Net-(D62-Pad1) -> col10
- SW_DOWN1 pad 1: col13 -> Net-(D73-K)
- SW_DOWN1 pad 2: Net-(D73-Pad1) -> col13
- SW_E1 pad 1: col3 -> Net-(D20-K)
- SW_E1 pad 2: Net-(D20-Pad1) -> col3
- SW_END1 pad 1: col14 -> Net-(D31-K)
- SW_END1 pad 2: Net-(D31-Pad1) -> col14
- SW_EQUAL1 pad 1: col12 -> Net-(D13-K)
- SW_EQUAL1 pad 2: Net-(D13-Pad1) -> col12
- SW_ESC1 pad 1: col0 -> Net-(D1-K)
- SW_ESC1 pad 2: Net-(D1-Pad1) -> col0
- SW_F1 pad 1: col4 -> Net-(D39-K)
- SW_F1 pad 2: Net-(D39-Pad1) -> col4
- SW_G1 pad 1: col5 -> Net-(D40-K)
- SW_G1 pad 2: Net-(D40-Pad1) -> col5
- SW_H1 pad 1: col6 -> Net-(D41-K)
- SW_H1 pad 2: Net-(D41-Pad1) -> col6
- SW_HOME1 pad 1: RotB -> Net-(D16-K)
- SW_HOME1 pad 2: Net-(D16-Pad1) -> RotB
- SW_I1 pad 1: col8 -> Net-(D25-K)
- SW_I1 pad 2: Net-(D25-Pad1) -> col8
- SW_ISO_ENT1 pad 1: col13 -> Net-(D46-K)
- SW_ISO_ENT1 pad 2: Net-(D46-Pad1) -> col13
- SW_ISO_\1 pad 1: col12 -> Net-(D45-K)
- SW_ISO_\1 pad 2: Net-(D45-Pad1) -> col12
- SW_J1 pad 1: col7 -> Net-(D42-K)
- SW_J1 pad 2: Net-(D42-Pad1) -> col7
- SW_K1 pad 1: col8 -> Net-(D43-K)
- SW_K1 pad 2: Net-(D43-Pad1) -> col8
- SW_L1 pad 1: col9 -> Net-(D44-K)
- SW_L1 pad 2: Net-(D44-Pad1) -> col9
- SW_LALT_1.25U1 pad 1: col1 -> Net-(D65-K)
- SW_LALT_1.25U1 pad 2: Net-(D65-Pad1) -> col1
- SW_LCMD_1.25U1 pad 1: col2 -> Net-(D66-K)
- SW_LCMD_1.25U1 pad 2: Net-(D66-Pad1) -> col2
- SW_LCTRL_1.25U1 pad 1: col0 -> Net-(D64-K)
- SW_LCTRL_1.25U1 pad 2: Net-(D64-Pad1) -> col0
- SW_LEFT1 pad 1: col12 -> Net-(D72-K)
- SW_LEFT1 pad 2: Net-(D72-Pad1) -> col12
- SW_LSQBR1 pad 1: col11 -> Net-(D28-K)
- SW_LSQBR1 pad 2: Net-(D28-Pad1) -> col11
- SW_M1 pad 1: col8 -> Net-(D60-K)
- SW_M1 pad 2: Net-(D60-Pad1) -> col8
- SW_MINUS1 pad 1: col11 -> Net-(D12-K)
- SW_MINUS1 pad 2: Net-(D12-Pad1) -> col11
- SW_N1 pad 1: col7 -> Net-(D59-K)
- SW_N1 pad 2: Net-(D59-Pad1) -> col7
- SW_O1 pad 1: col9 -> Net-(D26-K)
- SW_O1 pad 2: Net-(D26-Pad1) -> col9
- SW_P1 pad 1: col10 -> Net-(D27-K)
- SW_P1 pad 2: Net-(D27-Pad1) -> col10
- SW_PGDN1 pad 1: col14 -> Net-(D63-K)
- SW_PGDN1 pad 2: Net-(D63-Pad1) -> col14
- SW_PGUP1 pad 1: col14 -> Net-(D47-K)
- SW_PGUP1 pad 2: Net-(D47-Pad1) -> col14
- SW_Q1 pad 1: col1 -> Net-(D18-K)
- SW_Q1 pad 2: Net-(D18-Pad1) -> col1
- SW_QUOTE1 pad 1: col11 -> Net-(D33-K)
- SW_QUOTE1 pad 2: Net-(D33-Pad1) -> col11
- SW_R1 pad 1: col4 -> Net-(D21-K)
- SW_R1 pad 2: Net-(D21-Pad1) -> col4
- SW_RIGHT1 pad 1: col14 -> Net-(D74-K)
- SW_RIGHT1 pad 2: Net-(D74-Pad1) -> col14
- SW_RSHIFT1 pad 1: col12 -> Net-(D50-K)
- SW_RSHIFT1 pad 2: Net-(D50-Pad1) -> col12
- SW_RSQBR1 pad 1: col12 -> Net-(D29-K)
- SW_RSQBR1 pad 2: Net-(D29-Pad1) -> col12
- SW_R_CMD1 pad 1: col10 -> Net-(D70-K)
- SW_R_CMD1 pad 2: Net-(D70-Pad1) -> col10
- SW_R_CTRL_1.25U1 pad 1: col11 -> Net-(D71-K)
- SW_R_CTRL_1.25U1 pad 2: Net-(D71-Pad1) -> col11
- SW_S1 pad 1: col2 -> Net-(D37-K)
- SW_S1 pad 2: Net-(D37-Pad1) -> col2
- SW_SEMICOLON1 pad 1: col10 -> Net-(D34-K)
- SW_SEMICOLON1 pad 2: Net-(D34-Pad1) -> col10
- SW_SPL_SPACE_L1 pad 1: col4 -> Net-(D67-K)
- SW_SPL_SPACE_L1 pad 2: Net-(D67-Pad1) -> col4
- SW_SPL_SPACE_M1 pad 2: Net-(D68-Pad1) -> Net-(D68-K)
- SW_SPL_SPACE_R1 pad 1: col8 -> Net-(D69-K)
- SW_SPL_SPACE_R1 pad 2: Net-(D69-Pad1) -> col8
- SW_T1 pad 1: col5 -> Net-(D22-K)
- SW_T1 pad 2: Net-(D22-Pad1) -> col5
- SW_TAB1 pad 1: col0 -> Net-(D17-K)
- SW_TAB1 pad 2: Net-(D17-Pad1) -> col0
- SW_U1 pad 1: col7 -> Net-(D24-K)
- SW_U1 pad 2: Net-(D24-Pad1) -> col7
- SW_UP1 pad 1: col13 -> Net-(D51-K)
- SW_UP1 pad 2: Net-(D51-Pad1) -> col13
- SW_V1 pad 1: col5 -> Net-(D57-K)
- SW_V1 pad 2: Net-(D57-Pad1) -> col5
- SW_W1 pad 1: col2 -> Net-(D19-K)
- SW_W1 pad 2: Net-(D19-Pad1) -> col2
- SW_X1 pad 1: col3 -> Net-(D55-K)
- SW_X1 pad 2: Net-(D55-Pad1) -> col3
- SW_Y1 pad 1: col6 -> Net-(D23-K)
- SW_Y1 pad 2: Net-(D23-Pad1) -> col6
- SW_Z1 pad 1: col2 -> Net-(D54-K)
- SW_Z1 pad 2: Net-(D54-Pad1) -> col2
- U1 pad 22: unconnected-(U1-Pad22) -> /rst
- U1 pad 24: unconnected-(U1-Pad24) -> /Vbat
- U2 pad 4: GND -> mux3
- U2 pad 5: mux3 -> GND
Routing:
- net Net-(D73-Pad1): track 162.7 -> 0.00 mm
- net Net-(D74-Pad1): track 158.3 -> 0.00 mm
- net Net-(D64-Pad1): track 158.0 -> 0.00 mm
- net Net-(D74-K): track 0.00 -> 153.9 mm, vias 0 -> 1
- net Net-(D64-K): track 0.00 -> 149.0 mm, vias 0 -> 1
- net Net-(D51-Pad1): track 142.9 -> 0.00 mm
- net Net-(D73-K): track 0.00 -> 138.3 mm, vias 0 -> 1
- net Net-(D71-Pad1): track 137.8 -> 0.00 mm
- net Net-(D63-Pad1): track 135.8 -> 0.00 mm
- net Net-(D66-K): track 0.00 -> 133.5 mm, vias 0 -> 1
- net Net-(D71-K): track 0.00 -> 133.4 mm, vias 0 -> 1
- net Net-(D46-Pad1): track 133.2 -> 0.00 mm
- net Net-(D66-Pad1): track 132.3 -> 0.00 mm
- net Net-(D72-Pad1): track 129.9 -> 0.00 mm
- net Net-(D63-K): track 0.00 -> 129.9 mm, vias 0 -> 1
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Other:
- board text removed: "1.5U \"
- board text removed: "1U"
- board text removed: "2.25U ENTER"
- board text removed: "2.25U SHIFT"
- board text removed: "6.25U"
- board text removed: "JLCJLCJLCJLC"
- board text removed: "SPACE"

Commit message: Add alternative LEDs instead of OLED
Parts:
- removed D14, D30: 1N4148, lagom:D_MiniMELF_noSilk
- added D75: red, LED_SMD:LED_1206_3216Metric, F.Cu at (294.0, 50.4)
- added D76: green, LED_SMD:LED_1206_3216Metric, F.Cu at (289.0, 55.3)
- added R1: 680R, Resistor_SMD:R_1206_3216Metric, F.Cu at (291.5, 52.9)
- added R2: 680R, Resistor_SMD:R_1206_3216Metric, F.Cu at (296.5, 48.1)
- moved D15 6.75 mm to (279.3, 52.9)
- moved D73 6.75 mm to (267.4, 52.9)
- moved D31 6.75 mm to (276.9, 50.5)
- moved D51 6.75 mm to (265.0, 55.3)
- moved D46 6.75 mm to (262.6, 57.7)
- moved D47 6.75 mm to (274.5, 48.2)
- moved D48 6.75 mm to (286.5, 57.7)
- moved D16 5.34 mm to (281.7, 55.3)
- moved D74 5.34 mm to (269.8, 50.5)
- moved D32 5.34 mm to (284.1, 57.7)
- moved D63 5.34 mm to (272.2, 48.2)
- moved D72 5.34 mm to (260.2, 57.7)
Routing:
- net SDA: track 257.6 -> 285.5 mm
- net row0: track 334.6 -> 308.1 mm
- net row1: track 309.3 -> 292.3 mm, vias 16 -> 15
- net VCC: track 355.9 -> 372.6 mm, vias 4 -> 6
- net SCL: track 253.2 -> 264.7 mm
- net Net-(D16-K): track 74.4 -> 83.9 mm
- net Net-(D72-K): track 124.2 -> 132.0 mm
- net Net-(D47-K): track 117.3 -> 124.3 mm
- net RotA: track 43.0 -> 49.7 mm
- net Net-(D63-K): track 129.9 -> 136.3 mm
- net RotC: track 60.5 -> 66.3 mm
- net Net-(D31-K): track 88.6 -> 93.2 mm
- net Net-(D75-A): track 0.00 -> 4.39 mm
- net row4: track 264.6 -> 260.2 mm, vias 11 -> 10
- net Net-(D15-K): track 48.8 -> 52.9 mm
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
Commit message: Add signature
Other:
- board text added: "lagom modified by Tim Lauber"
- board text removed: "lagom v1"
Changed lines of the file:
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@@
 		(tags "capacitor")
 		(property "Reference" "C2"
-			(at 0 1.6 360)
+			(at 0 1.6 0)
 			(layer "F.SilkS")
 			(effects
@@
 		)
 		(property "Value" "0.1uF"
-			(at 0 1.68 360)
+			(at 0 1.68 0)
 			(layer "F.Fab")
 			(effects
@@
 		)
 		(fp_text user "${REFERENCE}"
-			(at 0 0 360)
+			(at 0 0 0)
 			(layer "F.Fab")
 			(effects
@@
 		(tags "rotary encoder")
 		(property "Reference" "SW83"
-			(at 2.8 -4.7 270)
+			(at 2.8 -4.7 -90)
 			(layer "F.SilkS")
 			(hide yes)
@@
 		(tags "rotary encoder")
 		(property "Reference" "SW84"
-			(at 2.8 -4.7 270)
+			(at 2.8 -4.7 -90)
 			(layer "F.SilkS")
 			(hide yes)
@@
 		)
 		(property "Value" "0.1uF"
-			(at 0 1.68 360)
+			(at 0 1.68 0)
 			(layer "F.Fab")
 			(effects
@@
 		)
 		(fp_text user "${REFERENCE}"
-			(at 0 0 360)
+			(at 0 0 0)
 			(layer "F.Fab")
 			(effects
@@
 		)
 	)
-	(gr_text "lagom v1"
-		(at 205.3 59.1 0)
+	(gr_text "lagom\nmodified\nby Tim Lauber"
+		(at 205.3 57.1 0)
 		(layer "F.SilkS")
 		(effects
