File: PCB/lagom_base/lagom_base.kicad_pcb (KiCad board)
At the start: 2 copper layers, 319.9 x 128.9 mm, 14 parts

Commit message: Change mounting equipment to M3 Hole + SMSI solder nuts
Parts:
- REF** (x9): value MountingHole_2.2mm_M2 -> MountingHole_3.2mm_M3; footprint MountingHole:MountingHole_2.2mm_M2 -> MountingHole:MountingHole_3.2mm_M3
Other:
- board text removed: "JLCJLCJLCJLC"

Commit message: Add signature
Parts:
- removed ? (x2): , 
Other:
- board text added: "STHLM KB lagom v1 design by mohoyt modified by Tim Lauber"
- board text removed: "STHLM KB lagom v1 design by mohoyt"
Changed lines of the file:
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@@
 		)
 	)
-	(footprint ""
-		(layer "F.Cu")
-		(at 52.525 186.225)
-		(property "Reference" ""
-			(at 0 0 0)
-			(layer "F.SilkS")
-			(effects
-				(font
-					(size 1.27 1.27)
-					(thickness 0.15)
-				)
-			)
-		)
-		(property "Value" ""
-			(at 0 0 0)
-			(layer "F.SilkS")
-			(effects
-				(font
-					(size 1.27 1.27)
-					(thickness 0.15)
-				)
-			)
-		)
-		(property "Footprint" ""
-			(at 0 0 0)
-			(layer "F.Fab")
-			(hide yes)
-			(effects
-				(font
-					(size 1.27 1.27)
-					(thickness 0.15)
-				)
-			)
-		)
-		(property "Datasheet" ""
-			(at 0 0 0)
-			(layer "F.Fab")
-			(hide yes)
-			(effects
-				(font
-					(size 1.27 1.27)
-					(thickness 0.15)
-				)
-			)
-		)
-		(property "Description" ""
-			(at 0 0 0)
-			(layer "F.Fab")
-			(hide yes)
-			(effects
-				(font
-					(size 1.27 1.27)
-					(thickness 0.15)
-				)
-			)
-		)
-		(pad "" np_thru_hole circle
-			(at 0 0)
-			(size 2.2 2.2)
-			(drill 2.2)
-			(layers "*.Cu" "*.Mask")
-		)
-	)
 	(footprint "MountingHole:MountingHole_3.2mm_M3"
 		(layer "F.Cu")
@@
 		)
 	)
-	(footprint ""
-		(layer "F.Cu")
-		(at 52.525 93.1125)
-		(property "Reference" ""
-			(at 0 0 0)
-			(layer "F.SilkS")
-			(effects
-				(font
-					(size 1.27 1.27)
-					(thickness 0.15)
-				)
-			)
-		)
-		(property "Value" ""
-			(at 0 0 0)
-			(layer "F.SilkS")
-			(effects
-				(font
-					(size 1.27 1.27)
-					(thickness 0.15)
-				)
-			)
-		)
-		(property "Footprint" ""
-			(at 0 0 0)
-			(layer "F.Fab")
-			(hide yes)
-			(effects
-				(font
-					(size 1.27 1.27)
-					(thickness 0.15)
-				)
-			)
-		)
-		(property "Datasheet" ""
-			(at 0 0 0)
-			(layer "F.Fab")
-			(hide yes)
-			(effects
-				(font
-					(size 1.27 1.27)
-					(thickness 0.15)
-				)
-			)
-		)
-		(property "Description" ""
-			(at 0 0 0)
-			(layer "F.Fab")
-			(hide yes)
-			(effects
-				(font
-					(size 1.27 1.27)
-					(thickness 0.15)
-				)
-			)
-		)
-		(pad "" np_thru_hole circle
-			(at 0 0)
-			(size 2.2 2.2)
-			(drill 2.2)
-			(layers "*.Cu" "*.Mask")
-		)
-	)
 	(footprint "MountingHole:MountingHole_3.2mm_M3"
 		(layer "F.Cu")
@@
 		(layer "Edge.Cuts")
 	)
-	(gr_text "STHLM KB lagom v1\ndesign by mohoyt"
+	(gr_text "STHLM KB lagom v1\ndesign by mohoyt\nmodified by Tim Lauber"
 		(at 207.7125 152.8 0)
 		(layer "F.SilkS")
