File: PCB/lagom_plate/lagom_plate.kicad_pcb (KiCad board)
At the start: 2 copper layers, 319.9 x 128.9 mm, 11 parts

Commit message: plate - Remove section for oled and rotary encoder.
Other:
- board size 319.9 x 128.9 mm -> 319.9 x 102.7 mm

Commit message: Cleanup outline
Parts:
- removed ? (x2): , 
Routing:
- net (no net): vias 3 -> 0
Other:
- outline, holes or cut-outs redrawn
- board text removed: "JLCJLCJLCJLC"

Commit message: Change mounting equipment to M3 Hole + SMSI solder nuts
Parts:
- REF** (x9): value MountingHole_2.2mm_M2 -> Mounting_Wuerth_WA-SMSI-M3_H3mm_9774030360; footprint MountingHole:MountingHole_2.2mm_M2 -> Mounting_Wuerth:Mounting_Wuerth_WA-SMSI-M3_H3mm_9774030360; moved to B.Cu
- turned REF** to 180 degrees (x9)

Commit message: Add signature
Other:
- board text added: "modified by Tim Lauber"
Changed lines of the file:
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@@
+		)
+	)
+	(gr_text "modified by Tim Lauber"
+		(at 198.7 127.1 0)
+		(layer "B.SilkS")
+		(effects
+			(font
+				(size 1 1)
+				(thickness 0.15)
+			)
+			(justify left bottom mirror)
 		)
 	)
